File: Kicad_MixtapeBarebone/Mixtape_Barebone.sch (KiCad schematic (older format))
At the start: 29 parts, among them IC1 ATTINY85-20PU, J1 PB5, J10 S-Out, J11 LED, J2 PB3, J3 PB4, J4 GND, J5 PB0, J6 PB1, J6 PB2, J8 VCC, J9 Prog, SW1 SW_SPST

Commit message: Designing the MicroCore Barebone Mixtape
Connections:
- net Prog: now reaches C1.1, IC1.2 (PB3(XTAL1/CLKI/OC1B/ADC3/PCINT3)), J2.1 (P1), R1.2, R2.1, R3.1
Changed lines of the file:
@@
 Wire Wire Line
 	5200 3950 5250 3950
+Text GLabel 3900 4150 3    60   Input ~ 0
+Prog
+Wire Wire Line
+	3900 4150 3900 3950
+Connection ~ 3900 3950
 $EndSCHEMATC

Commit message: mCore Mixtape and more DIY-CAD stuff
Parts:
- added NEO1, NEO2: SK6813b, 8BitMixtape_Stomp:Mixtape_NEO_WS2812B, symbol LED_Dual_ACAC
Connections:
- net GND: now also NEO1.3 (A2), NEO2.3 (A2)
- net VCC: now also NEO1.1 (A1), NEO2.1 (A1)
- net NEO: now reaches IC1.5 (PB0(MOSI/DI/SDA/AIN0/OC0A/OC1A/AREF/PCINT0)), J5.1 (P1)
- net NEO: now also NEO1.4 (K2)
- new net: NEO1.2 (K1), NEO2.4 (K2)
Changed lines of the file:
@@
 	3900 4150 3900 3950
 Connection ~ 3900 3950
+Text GLabel 5350 3350 2    60   Input ~ 0
+NEO
+Wire Wire Line
+	5350 3350 5250 3350
+Connection ~ 5250 3350
+Wire Wire Line
+	5650 4900 5800 4900
+Wire Wire Line
+	5650 4700 5800 4700
+$Comp
+L GND #PWR013
+U 1 1 5B5D688D
+P 5650 4900
+F 0 "#PWR013" H 5650 4650 50  0001 C CNN
+F 1 "GND" H 5650 4750 50  0000 C CNN
+F 2 "" H 5650 4900 50  0001 C CNN
+F 3 "" H 5650 4900 50  0001 C CNN
+	1    5650 4900
+	1    0    0    -1
+$EndComp
+$Comp
+L VCC #PWR014
+U 1 1 5B5D67EC
+P 5650 4700
+F 0 "#PWR014" H 5650 4550 50  0001 C CNN
+F 1 "VCC" H 5650 4850 50  0000 C CNN
+F 2 "" H 5650 4700 50  0001 C CNN
+F 3 "" H 5650 4700 50  0001 C CNN
+	1    5650 4700
+	1    0    0    -1
+$EndComp
+$Comp
+L LED_Dual_ACAC NEO2
+U 1 1 5B5D6689
+P 6100 4800
+F 0 "NEO2" H 6100 5025 50  0000 C CNN
+F 1 "SK6813b" H 6100 4550 50  0000 C CNN
+F 2 "8BitMixtape_Stomp:Mixtape_NEO_WS2812B" H 6130 4800 50  0001 C CNN
+F 3 "" H 6130 4800 50  0001 C CNN
+	1    6100 4800
+	1    0    0    -1
+$EndComp
+Wire Wire Line
+	6600 5600 6400 5600
+Text GLabel 6600 5600 2    60   Input ~ 0
+NEO
+Wire Wire Line
+	5650 5600 5800 5600
+Wire Wire Line
+	5650 5400 5800 5400
+$Comp
+L GND #PWR015
+U 1 1 5B5D71FF
+P 5650 5600
+F 0 "#PWR015" H 5650 5350 50  0001 C CNN
+F 1 "GND" H 5650 5450 50  0000 C CNN
+F 2 "" H 5650 5600 50  0001 C CNN
+F 3 "" H 5650 5600 50  0001 C CNN
+	1    5650 5600
+	1    0    0    -1
+$EndComp
+$Comp
+L VCC #PWR016
+U 1 1 5B5D7205
+P 5650 5400
+F 0 "#PWR016" H 5650 5250 50  0001 C CNN
+F 1 "VCC" H 5650 5550 50  0000 C CNN
+F 2 "" H 5650 5400 50  0001 C CNN
+F 3 "" H 5650 5400 50  0001 C CNN
+	1    5650 5400
+	1    0    0    -1
+$EndComp
+$Comp
+L LED_Dual_ACAC NEO1
+U 1 1 5B5D720B
+P 6100 5500
+F 0 "NEO1" H 6100 5725 50  0000 C CNN
+F 1 "SK6813b" H 6100 5250 50  0000 C CNN
+F 2 "8BitMixtape_Stomp:Mixtape_NEO_WS2812B" H 6130 5500 50  0001 C CNN
+F 3 "" H 6130 5500 50  0001 C CNN
+	1    6100 5500
+	1    0    0    -1
+$EndComp
+Wire Wire Line
+	6400 4900 6550 4900
+Wire Wire Line
+	6550 4900 6550 5400
+Wire Wire Line
+	6550 5400 6400 5400
 $EndSCHEMATC
